File: ModuleElectronice/ModulDistributiePutere/ModulDistributiePutere.sch (KiCad schematic (older format))
At the start: 24 parts

Commit message: Updated files + Documentation April 7 - 2019
Parts:
- added C?: 1100uF, symbol Device:CP
- added C?: 560uF, symbol Device:CP
- added C?: 2200uF, symbol Device:CP
- added C? (x2): 100nF, symbol Device:C
- added D? (x2): 1N4148, Diode_THT:D_DO-35_SOD27_P7.62mm_Horizontal, symbol Diode:1N4148
- added D?: LED, symbol Device:LED
- added Q?: 2N3904, Package_TO_SOT_THT:TO-92_Inline, symbol Transistor_BJT:2N3904
- added R?: 3K, symbol Device:R
- added R? (x4): 1K, symbol Device:R
- added U?: LM1085-5.0, symbol Regulator_Linear:LM1085-5.0
Connections:
- net labels added: D10, D11, D12, D13
- wire segments 81 -> 126
Other:
- note added: "Radiator extrudat: SK 09 20 SA TO 220\nTO220; neagră; \nL: 20mm; W: 29mm; H: 11,5mm; 15K/W"
- moved on the sheet: A?, Q?, R?

Commit message: Updated files
Parts:
- removed C?: 1100uF, symbol Device:CP
- removed C?: 100nF, symbol Device:C
- removed D? (x2): 1N4148, Diode_THT:D_DO-35_SOD27_P7.62mm_Horizontal, symbol Diode:1N4148
- removed D?: LED, symbol Device:LED
- removed R?: 3K, symbol Device:R
- removed R? (x2): 1K, symbol Device:R
- removed U?: LM1085-5.0, symbol Regulator_Linear:LM1085-5.0
- added C?: 470uF, symbol Device:CP
- added D3, D4, D5, D7: LED, LED_THT:LED_D5.0mm, symbol Device:LED
- added D?: MBR735, Package_TO_SOT_THT:TO-220-2_Vertical, symbol Diode:MBR735
- added L?: 33uF, symbol Device:L
- added R13, R14, R15, R16: 1K, Resistor_SMD:R_1206_3216Metric_Pad1.42x1.75mm_HandSolder, symbol Device:R
- added R?: 5K1, symbol Device:R
- added U?: LM2596S-5, Package_TO_SOT_SMD:TO-263-5_TabPin3, symbol Regulator_Switching:LM2596S-5
- C1: renamed from C?; footprint (none) -> Capacitor_THT:CP_Radial_D12.5mm_P5.00mm
- C2: renamed from C?; value 560uF -> 1100uF; footprint (none) -> Capacitor_THT:C_Radial_D12.5mm_H25.0mm_P5.00mm
- J1: renamed from J?; footprint (none) -> Connector_PinHeader_2.54mm:PinHeader_1x03_P2.54mm_Vertical
- R1, R17, R19, R4, R6, R8: renamed from R?; value R -> 1K; footprint (none) -> Resistor_SMD:R_1206_3216Metric_Pad1.42x1.75mm_HandSolder
- R10, R9: renamed from R?; footprint (none) -> Resistor_SMD:R_1206_3216Metric_Pad1.42x1.75mm_HandSolder
- R18, R2, R20: renamed from R?; value R -> 120; footprint (none) -> Resistor_THT:R_Axial_DIN0414_L11.9mm_D4.5mm_P25.40mm_Horizontal
- R3, R5, R7: renamed from R?; value R -> 9K; footprint (none) -> Resistor_SMD:R_1206_3216Metric_Pad1.42x1.75mm_HandSolder
- gave numbers to parts that had none: 13
Connections:
- net labels added: D6, D7, D8, D9
- wire segments 126 -> 137
Other:
- note added: "GREEN LED's"
- note added: "RED LED's"
- note added: "Status LED's\n"
- moved on the sheet: A1, C2, C3, Q2, R10, R3, R4, R5, R6, R7, R8, R9
